File: minRead_pcb.kicad_sch (KiCad schematic)
At the start: 118 parts, among them J1 USB_C_Receptacle, J2 FH34SRJ-24S-0.5SH_50_, J3 FH34SRJ-6S-0.5SH_50_, J5 Conn_01x02, J6 PPTC052LFBN-RC, J7 Micro_SD_Card, Q1 FS8205A, Q2 IRLML6402, Q3 IRLML6402, Q4 BSS138, Q5 BSS138, Q6 BSS138, Q7 IRLML6402, Q8 IRLML6402, Q9 MMBT3904, SW1 SW_Push, SW10 SW_Push, SW12 SW_Push, SW2 SW_Push, SW3 SW_Push, SW4 SW_Push, SW5 SW_Push, SW6 SW_Push, SW7 SW_Push, SW8 SW_Push, SW9 SW_Push, U1 TPD4E1U06DBVR, U2 AP3012, U3 AP2112K-3.3, U4 ESP32-S3-WROOM-1, U5 DW01A, U6 TPD4E1U06DBVR, U7 MCP73832-2-OT

Commit message: first draft for 1.0
Parts:
- removed J6: PPTC052LFBN-RC, PPTC_10:CONN_PPTC052LFBN-RC_SUL, symbol PPTC_10:PPTC052LFBN-RC
- removed SW12: SW_Push, Button_Switch_SMD:SW_SPST_PTS810, symbol Switch:SW_Push
- removed TP1, TP3, TP5, TP7: TestPoint, TestPoint:TestPoint_THTPad_1.0x1.0mm_Drill0.5mm, symbol Connector:TestPoint
- removed U2: AP3012, Package_TO_SOT_SMD:SOT-23-5, symbol Regulator_Switching:AP3012
- added CR2: TSD05CDYFR, Diode_SMD:D_SOD-323_HandSoldering, symbol TSD05CDYFR:TSD05CDYFR
- added D3: SMAJ30A, Diode_SMD:D_SMA, symbol Diode:SMAJ30A
- added D8: PESD2IVN-UX, Package_TO_SOT_SMD:SOT-323_SC-70_Handsoldering, symbol Device:D_TVS_Dual_ACA
- added H5, H6: MountingHole_Pad, MountingHole:MountingHole_2.2mm_M2_DIN965_Pad_TopBottom, symbol Mechanical:MountingHole_Pad
- added J6: PPPC062LJBN-RC, PPPC_12:CONN_PPPC062LJBN-RC_SUL, symbol PPPC_12:PPPC062LJBN-RC
- added SW11: SW_Push, mjtp1117:MJTP1117, symbol Switch:SW_Push
- added U2: LM27313XMF, Package_TO_SOT_SMD:SOT-23-5, symbol Regulator_Switching:LM27313XMF
- added U8, U9: TPD4E1U06DBVR, Package_TO_SOT_SMD:SOT-23-6_Handsoldering, symbol TPD4E1U06DBVR:TPD4E1U06DBVR
- CR1: footprint footprints:TVS_SOD2_DYF_TEX-M -> Diode_SMD:D_SOD-323_HandSoldering
- L1, L2: value 10u -> 22u
- Q2, Q3, Q7, Q8: value IRLML6402 -> AO3419
- SW1, SW10, SW4, SW5, SW7: footprint Button_Switch_THT:SW_Tactile_SPST_Angled_PTS645Vx39-2LFS -> mjtp1117:MJTP1117
- SW2, SW3, SW8, SW9: footprint Button_Switch_SMD:SW_SPST_PTS810 -> mjtp1117:MJTP1117
- SW6: footprint Button_Switch_SMD:SW_SPST_PTS810 -> Button_Switch_THT:SW_PUSH_6mm
Connections:
- net 3V3: now also SW10.2, CR2.1 (I/O), J6.12; no longer SW10.1
- net C-: now also D8.1 (A1), J6.2
- net ESP32_EN: now also SW11.2
- net GND: now also CR2.2 (GND), D3.2 (A2), D8.2 (common), H5.1, H6.1, J6.1, SW11.1, U2.2 (GND), U8.2, U9.2
- net LED_SW: now also D3.1 (A1), J6.7
- net PWM_LED: now also U2.4 (EN)
- net PWR_BUTTON: now also SW10.1; no longer SW10.2
- net UNUSED_GPIO_15: now also J6.5, U9.3
- net UNUSED_GPIO_16: now also J6.10, U9.6
- net UNUSED_GPIO_45: now also J6.3, U9.1
- net UNUSED_GPIO_46: now also J6.9, U8.6
- net UNUSED_GPIO_47: now also J6.4, U8.1
- net W-: now also D8.3 (A2), J6.8
- net at D7.2 (A), L2.2: now also U2.1 (SW)
- net at C12.2, L2.1, Q7.3 (D): now also U2.5 (VIN)
- net at Q5.2 (S), Q6.2 (S), R37.1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: now also U2.3 (FB)
- net RX: now reaches U4.36 (RXD0)
- net RX: now also J6.6, U9.4
- net TX: now reaches U4.37 (TXD0)
- net TX: now also J6.11, U8.3
- net BACK: no longer names the net of R20.1, SW9.2
- net CONFIRM: no longer names the net of R19.1, SW8.2
- net LEFT: no longer names the net of R18.1, SW3.2
- no-connect marks 14 -> 13
Other:
- note added: "External Peripheral ESD Protection"
- note added: "NR3015T220MNGH"
- note removed: "External Buttons"
- note removed: "SRN3010C-100m"

Commit message: update silkscreen
Parts:
- SW6: now not fitted
Changed lines of the file:
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@@
 		(in_bom yes)
 		(on_board yes)
-		(dnp no)
+		(dnp yes)
 		(fields_autoplaced yes)
 		(property "Reference" "SW6"

Commit message: revised layout for emi/emc
Changed lines of the file:
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@@
 	(text "LDO 3.3V"
 		(exclude_from_sim no)
-		(at 162.56 25.146 0)
+		(at 172.212 25.654 0)
 		(effects
 			(font

Commit message: added fuse changed mbr to b5819w for current rating increase changed r38 to reduce leakage spiffied up silkscreen
Parts:
- added F1: 0805L100WR, Fuse:Fuse_0805_2012Metric_Pad1.15x1.40mm_HandSolder, symbol Device:Polyfuse
- D1, D2, D4, D5, D6: value MBR0530 -> B5819W
- D7: value MBR0540 -> B5819W
- R38: value 100k -> 10k
Connections:
- net VBUS_PRE: now also F1.1; no longer D1.2 (A)
- new net: D1.2 (A), F1.2
Other:
- moved on the sheet: D1
Changed lines of the file:
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@@
 	)
 	(junction
+		(at 67.31 30.48)
+		(diameter 0)
+		(color 0 0 0 0)
+	)
+	(junction
 		(at 52.07 163.83)
 		(diameter 0)
@@
 	)
 	(junction
+		(at 48.26 30.48)
+		(diameter 0)
+		(color 0 0 0 0)
+	)
+	(junction
 		(at 420.37 55.88)
 		(diameter 0)
@@
 	)
 	(junction
-		(at 62.23 30.48)
-		(diameter 0)
-		(color 0 0 0 0)
-	)
-	(junction
 		(at 431.8 63.5)
 		(diameter 0)
@@
 	(wire
 		(pts
-			(xy 52.07 30.48) (xy 48.26 30.48)
-		)
-		(stroke
-			(width 0)
-			(type default)
-		)
-	)
-	(wire
-		(pts
 			(xy 148.59 323.85) (xy 115.57 323.85)
 		)
@@
 	(wire
 		(pts
+			(xy 49.53 30.48) (xy 48.26 30.48)
+		)
+		(stroke
+			(width 0)
+			(type default)
+		)
+	)
+	(wire
+		(pts
 			(xy 50.8 156.21) (xy 55.88 156.21)
 		)
@@
 	(wire
 		(pts
+			(xy 57.15 30.48) (xy 58.42 30.48)
+		)
+		(stroke
+			(width 0)
+			(type default)
+		)
+	)
+	(wire
+		(pts
 			(xy 373.38 182.88) (xy 373.38 186.69)
 		)
@@
 	(wire
 		(pts
-			(xy 59.69 30.48) (xy 62.23 30.48)
+			(xy 66.04 30.48) (xy 67.31 30.48)
 		)
 		(stroke
@@
 	(wire
 		(pts
+			(xy 67.31 25.4) (xy 67.31 30.48)
+		)
+		(stroke
+			(width 0)
+			(type default)
+		)
+	)
+	(wire
+		(pts
 			(xy 52.07 279.4) (xy 58.42 279.4)
 		)
@@
 	(wire
 		(pts
+			(xy 67.31 30.48) (xy 68.58 30.48)
+		)
+		(stroke
+			(width 0)
+			(type default)
+		)
+	)
+	(wire
+		(pts
 			(xy 148.59 325.12) (xy 148.59 327.66)
 		)
@@
 	(wire
 		(pts
-			(xy 62.23 30.48) (xy 68.58 30.48)
-		)
-		(stroke
-			(width 0)
-			(type default)
-		)
-	)
-	(wire
-		(pts
 			(xy 334.01 274.32) (xy 339.09 274.32)
 		)
@@
 	(wire
 		(pts
+			(xy 48.26 24.13) (xy 48.26 30.48)
+		)
+		(stroke
+			(width 0)
+			(type default)
+		)
+	)
+	(wire
+		(pts
 			(xy 66.04 284.48) (xy 66.04 288.29)
 		)
@@
 	)
 	(label "VBUS_PRE"
-		(at 49.53 30.48 90)
+		(at 48.26 24.13 180)
 		(effects
 			(font
 				(size 1.27 1.27)
 			)
-			(justify left bottom)
+			(justify right bottom)
 		)
 	)
@@
 			)
 		)
-		(property "Value" "MBR0540"
+		(property "Value" "B5819W"
 			(at 325.4375 270.51 0)
 			(effects
@@
 	(symbol
 		(lib_id "power:PWR_FLAG")
-		(at 62.23 30.48 0)
+		(at 67.31 25.4 0)
 		(unit 1)
 		(exclude_from_sim no)
@@
 		(fields_autoplaced yes)
 		(property "Reference" "#FLG01"
-			(at 62.23 28.575 0)
+			(at 67.31 23.495 0)
 			(effects
 				(font
@@
 		)
 		(property "Value" "PWR_FLAG"
-			(at 62.23 25.4 0)
+			(at 67.31 20.32 0)
 			(effects
 				(font
@@
 		)
 		(property "Footprint" ""
-			(at 62.23 30.48 0)
+			(at 67.31 25.4 0)
 			(effects
 				(font
@@
 		)
 		(property "Datasheet" "~"
-			(at 62.23 30.48 0)
+			(at 67.31 25.4 0)
 			(effects
 				(font
@@
 		)
 		(property "Description" "Special symbol for telling ERC where power comes from"
-			(at 62.23 30.48 0)
+			(at 67.31 25.4 0)
 			(effects
 				(font
@@
 	(symbol
 		(lib_id "Diode:MBR0530")
-		(at 55.88 30.48 180)
+		(at 62.23 30.48 180)
 		(unit 1)
 		(exclude_from_sim no)
@@
 		(on_board yes)
 		(dnp no)
-		(fields_autoplaced yes)
 		(property "Reference" "D1"
-			(at 56.1975 24.13 0)
+			(at 62.738 24.892 0)
 			(effects
 				(font
@@
 			)
 		)
-		(property "Value" "MBR0530"
-			(at 56.1975 26.67 0)
+		(property "Value" "B5819W"
+			(at 63.246 27.178 0)
 			(effects
 				(font
@@
 		)
 		(property "Footprint" "Diode_SMD:D_SOD-123"
-			(at 55.88 26.035 0)
+			(at 62.23 26.035 0)
 			(effects
 				(font
@@
 		)
 		(property "Datasheet" "http://www.mccsemi.com/up_pdf/MBR0520~MBR0580(SOD123).pdf"
-			(at 55.88 30.48 0)
+			(at 62.23 30.48 0)
 			(effects
 				(font
@@
 		)
 		(property "Description" "30V 0.5A Schottky Power Rectifier Diode, SOD-123"
-			(at 55.88 30.48 0)
+			(at 62.23 30.48 0)
 			(effects
 				(font
@@
 			)
 		)
-		(property "Value" "MBR0530"
+		(property "Value" "B5819W"
 			(at 68.58 306.3874 90)
 			(effects
@@
 			)
 		)
-		(property "Value" "MBR0530"
+		(property "Value" "B5819W"
 			(at 52.07 305.7524 90)
 			(effects
@@
 			)
 		)
-		(property "Value" "100k"
+		(property "Value" "10k"
 			(at 125.73 62.2299 0)
 			(effects
@@
 			)
 		)
-		(property "Value" "MBR0530"
+		(property "Value" "B5819W"
 			(at 131.1275 49.53 0)
 			(effects
@@
 	)
 	(symbol
+		(lib_id "Device:Polyfuse")
+		(at 53.34 30.48 90)
+		(unit 1)
+		(exclude_from_sim no)
+		(in_bom yes)
+		(on_board yes)
+		(dnp no)
+		(fields_autoplaced yes)
+		(property "Reference" "F1"
+			(at 53.34 24.13 90)
+			(effects
+				(font
+					(size 1.27 1.27)
+				)
+			)
+		)
+		(property "Value" "0805L100WR"
+			(at 53.34 26.67 90)
+			(effects
+				(font
+					(size 1.27 1.27)
+				)
+			)
+		)
+		(property "Footprint" "Fuse:Fuse_0805_2012Metric_Pad1.15x1.40mm_HandSolder"
+			(at 58.42 29.21 0)
+			(effects
+				(font
+					(size 1.27 1.27)
+				)
+				(justify left)
+				(hide yes)
+			)
+		)
+		(property "Datasheet" "~"
+			(at 53.34 30.48 0)
+			(effects
+				(font
+					(size 1.27 1.27)
+				)
+				(hide yes)
+			)
+		)
+		(property "Description" "Resettable fuse, polymeric positive temperature coefficient"
+			(at 53.34 30.48 0)
+			(effects
+				(font
+					(size 1.27 1.27)
+				)
+				(hide yes)
+			)
+		)
+		(pin "1"
+		)
+		(pin "2"
+		)
+		(instances
+			(project ""
+				(path "/2fbd4c8f-b784-4d80-b374-4947df99a9bf"
+					(reference "F1")
+					(unit 1)
+				)
+			)
+		)
+	)
+	(symbol
 		(lib_id "TSD05CDYFR:TSD05CDYFR")
 		(at 36.83 124.46 0)
@@
 			)
 		)
-		(property "Value" "MBR0530"
+		(property "Value" "B5819W"
 			(at 38.1 305.1174 90)
 			(effects
