File: minRead_pcb.kicad_sch (KiCad schematic)
At the start: 122 parts, among them J1 USB_C_Receptacle, J2 FH34SRJ-24S-0.5SH_50_, J3 FH34SRJ-6S-0.5SH_50_, J5 Conn_01x02, J6 PPPC062LJBN-RC, J7 Micro_SD_Card, Q1 FS8205A, Q2 AO3419, Q3 AO3419, Q4 BSS138, Q5 BSS138, Q6 BSS138, Q7 AO3419, Q8 AO3419, Q9 MMBT3904, SW1 SW_Push, SW10 SW_Push, SW11 SW_Push, SW2 SW_Push, SW3 SW_Push, SW4 SW_Push, SW5 SW_Push, SW6 SW_Push, SW7 SW_Push, SW8 SW_Push, SW9 SW_Push, U1 TPD4E1U06DBVR, U2 LM27313XMF, U3 AP2112K-3.3, U4 ESP32-S3-WROOM-1, U5 DW01A, U6 TPD4E1U06DBVR, U7 MCP73832-2-OT, U8 TPD4E1U06DBVR, U9 TPD4E1U06DBVR

Commit message: shaved down dev header size
Parts:
- removed H5, H6: MountingHole_Pad, MountingHole:MountingHole_2.2mm_M2_DIN965_Pad_TopBottom, symbol Mechanical:MountingHole_Pad

Commit message: revised schematic/layout and LED driver sim; drop tracked sim raw output
Parts:
- removed Q9: MMBT3904, Package_TO_SOT_SMD:SOT-23_Handsoldering, symbol Transistor_BJT:MMBT3904
- added C21: 1n, Capacitor_SMD:C_0805_2012Metric_Pad1.18x1.45mm_HandSolder, symbol Device:C
- added C23: 100n, Capacitor_SMD:C_0805_2012Metric_Pad1.18x1.45mm_HandSolder, symbol Device:C
- added C24: 2.2n, Capacitor_SMD:C_0805_2012Metric_Pad1.18x1.45mm_HandSolder, symbol Device:C
- added D9: BZT52C22, Diode_SMD:D_SOD-123F, symbol Diode:BZT52Bxx
- added Q12, Q13, Q17: MMBT3904, Package_TO_SOT_SMD:SOT-23_Handsoldering, symbol Transistor_BJT:MMBT3904
- added Q14: AO3419, Package_TO_SOT_SMD:SOT-23_Handsoldering, symbol Transistor_FET:IRLML6402
- added Q15, Q16: MMBT3906, Package_TO_SOT_SMD:SOT-23_Handsoldering, symbol Transistor_BJT:MMBT3906
- added Q9: BSS138, Package_TO_SOT_SMD:SOT-23, symbol Transistor_FET:BSS138
- added R17, R49, R50: 1M, Resistor_SMD:R_0805_2012Metric_Pad1.20x1.40mm_HandSolder, symbol Device:R
- added R42: 330, Resistor_SMD:R_0805_2012Metric_Pad1.20x1.40mm_HandSolder, symbol Device:R
- added R43: 22k, Resistor_SMD:R_0805_2012Metric_Pad1.20x1.40mm_HandSolder, symbol Device:R
- added R44, R45: 10k, Resistor_SMD:R_0805_2012Metric_Pad1.20x1.40mm_HandSolder, symbol Device:R
- added R46: 47k', Resistor_SMD:R_0805_2012Metric_Pad1.20x1.40mm_HandSolder, symbol Device:R
- added R47, R48: 18k, Resistor_SMD:R_0805_2012Metric_Pad1.20x1.40mm_HandSolder, symbol Device:R
- R39: value 10k -> 100k
- R41: value 10k -> 4.7k
- U2: value LM27313XMF -> AP3012
Connections:
- net 3V3: now also R39.2, Q14.2 (S), Q16.2 (E), R17.1; no longer R41.1
- net C-: now also R50.1
- net COOL_TOGGLE: no longer Q5.1 (G)
- net GND: now also C21.1, C23.2, C24.2, Q12.2 (E), Q13.2 (E), Q17.2 (E), R17.2, R49.2, R50.2
- net LED_PWR: no longer Q7.1 (G), R40.1
- net LED_SENSE: no longer R41.2
- net LED_SW: now also R41.2
- net W-: now also R49.1
- net WARM_TOGGLE: no longer Q6.1 (G)
- net at Q5.2 (S), Q6.2 (S), R37.1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: no longer R39.2
- net at R39.1: now also Q9.2 (S)
- new net: Q12.3 (C), Q9.1 (G), R42.2, R43.2
- new net: Q7.1 (G), Q9.3 (D), R40.1
- new net: Q15.1 (B), R45.2, R46.1
- new net: Q15.3 (C), R44.2
- new net: D9.1 (K), R41.1
- new net: Q17.1 (B), R48.2
- new net: Q13.1 (B), R43.1
- new net: Q16.1 (B), R47.2
- new net COLOR_SEL: Q5.1 (G), R47.1, R48.1
- new net COLOR_SEL_INV: C24.1, Q16.3 (C), Q17.3 (C), Q6.1 (G)
- new net ISO_GATE: R45.1
- new net LATCH_PWR: C23.1, Q14.3 (D), Q15.2 (E), R42.1, R46.2
- new net SENSE_N: C21.2, D9.2 (A), Q12.1 (B), R44.1
Other:
- moved on the sheet: C12, C9, D7, H1, H2, H3, H4, J3, L2, Q5, Q6, Q7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

Commit message: updated schematic with new LED circuit, new power path, new protections, esd fix ups, etc. resetting layout, will do later
Parts:
- removed D2: B5819W, Diode_SMD:D_SOD-123, symbol Diode:MBR0530
- removed Q2: AO3419, Package_TO_SOT_SMD:SOT-23_Handsoldering, symbol Transistor_FET:IRLML6402
- removed U2: AP3012, Package_TO_SOT_SMD:SOT-23-5, symbol Regulator_Switching:LM27313XMF
- added C25, C26: 1u, Capacitor_SMD:C_0805_2012Metric_Pad1.18x1.45mm_HandSolder, symbol Device:C
- added C27, C28, C29: 2.2n, Capacitor_SMD:C_0805_2012Metric_Pad1.18x1.45mm_HandSolder, symbol Device:C
- added D2: LED, LED_THT:LED_D3.0mm, symbol Device:LED
- added J4: FH34SRJ-6S-0.5SH_50_, FH34SRJ-6S-0.5SH(50):HRS_FH34SRJ-6S-0.5SH_50_, symbol FH34SRJ-6S-0.5SH(50):FH34SRJ-6S-0.5SH_50_
- added R51, R57, R58: 100k, Resistor_SMD:R_0805_2012Metric_Pad1.20x1.40mm_HandSolder, symbol Device:R
- added R52: 22k, Resistor_SMD:R_0805_2012Metric_Pad1.20x1.40mm_HandSolder, symbol Device:R
- added R56, R59: 1k, Resistor_SMD:R_0805_2012Metric_Pad1.20x1.40mm_HandSolder, symbol Device:R
- added R60, R61: 100, Resistor_SMD:R_0805_2012Metric_Pad1.20x1.40mm_HandSolder, symbol Device:R
- added U10: AP3031KTR, Package_TO_SOT_SMD:SOT-23-6_Handsoldering, symbol AP3031:AP3031KTR
- added U2: TPS2116DRL, Package_TO_SOT_SMD:SOT-583-8, symbol Power_Management:TPS2116DRL
- R37: value 82 -> 13.3
- R38: value 10k -> 310k
Connections:
- net 3V3: now also J4.2, R58.2
- net B+: now also R57.2
- net B-: now also R56.2; no longer Q3.1 (G)
- net BUTTON_ADC_1: now also C27.2, R60.2; no longer SW2.2
- net BUTTON_ADC_2: now also C28.2, R61.2; no longer SW1.2
- net CHG_STATUS: no longer U7.1 (STAT)
- net GND: now also C25.1, C26.2, C27.1, C28.1, C29.1, J4.1, J4.S1 (SHIELD), J4.S2 (SHIELD), R51.2, R52.1, U10.2 (GND), U2.1 (GND); no longer R38.2
- net LDO_IN: now also U2.2 (VOUT), U2.7 (VOUT)
- net LED_SW: now also U10.5 (OV)
- net P+: now also C26.1, U2.6 (VIN2)
- net PWM_LED: now also U10.4 (CTRL)
- net USB_VBUS: now also C25.2, D2.2 (A), U2.3 (VIN1), U2.5 (MODE)
- net 3031_SW: now reaches D7.2 (A), L2.2
- net 3031_SW: now also U10.1 (SW)
- net at C12.2, L2.1, Q7.3 (D): now also R52.2, U10.6 (V_{IN})
- net at Q5.2 (S), Q6.2 (S), R37.1: now also U10.3 (FB)
- net LED_ACTIVATE: now reaches Q13.3 (C)
- net LED_ACTIVATE: now also Q14.1 (G)
- net COOL_TOGGLE: no longer names the net of U4.7 (IO7)
- net LED_SENSE: no longer names the net of U4.11 (IO18)
- new net: D2.1 (K), R59.1
- new net: R59.2, U7.1 (STAT)
- new net: R60.1, SW2.2
- new net: R61.1, SW1.2
- new net: Q3.1 (G), R56.1, R57.1
- new net INT: J4.4
- new net PR1: R38.2, R51.1, U2.4 (PR1)
- new net RST: J4.3
- new net SCL: J4.6
- new net SDA: J4.5
- new net USB_STAT: R58.1, U2.8 (ST)
Other:
- note added: "2.5mA at 2.0Vf 4.6 - 2.0 / (0.0025) = 1kohm"
- note added: "Explanation for Q8:"
- note added: "HIGH = USB LOW = BATTERY"
- note added: "Switchover at ~4.1V"
- note added: "Touch Connector"
- note removed: "Explanation for Mosfet:"
- moved on the sheet: C12, C21, C23, C24, C32, C33, C36, C37, C4, C5, C6, C9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

Commit message: simplify led driver; assume frontlight always connected + other circuit component changes
Parts:
- removed C12, C9: 4.7u, Capacitor_SMD:C_0805_2012Metric_Pad1.18x1.45mm_HandSolder, symbol Device:C
- removed C21: 1n, Capacitor_SMD:C_0805_2012Metric_Pad1.18x1.45mm_HandSolder, symbol Device:C
- removed C23: 100n, Capacitor_SMD:C_0805_2012Metric_Pad1.18x1.45mm_HandSolder, symbol Device:C
- removed C24: 2.2n, Capacitor_SMD:C_0805_2012Metric_Pad1.18x1.45mm_HandSolder, symbol Device:C
- removed D7: B5819W, Diode_SMD:D_SOD-123, symbol Diode:MBR0540
- removed D9: BZT52C22, Diode_SMD:D_SOD-123F, symbol Diode:BZT52Bxx
- removed J4: FH34SRJ-6S-0.5SH_50_, FH34SRJ-6S-0.5SH(50):HRS_FH34SRJ-6S-0.5SH_50_, symbol FH34SRJ-6S-0.5SH(50):FH34SRJ-6S-0.5SH_50_
- removed L2: 22u, srn3010C-100m:IND_SRN3010C-100M, symbol Device:L
- removed Q12, Q13: MMBT3904, Package_TO_SOT_SMD:SOT-23_Handsoldering, symbol Transistor_BJT:MMBT3904
- removed Q14, Q7: AO3419, Package_TO_SOT_SMD:SOT-23_Handsoldering, symbol Transistor_FET:IRLML6402
- removed Q15: MMBT3906, Package_TO_SOT_SMD:SOT-23_Handsoldering, symbol Transistor_BJT:MMBT3906
- removed Q5, Q6, Q9: BSS138, Package_TO_SOT_SMD:SOT-23, symbol Transistor_FET:BSS138
- removed R17, R49, R50: 1M, Resistor_SMD:R_0805_2012Metric_Pad1.20x1.40mm_HandSolder, symbol Device:R
- removed R37: 13.3, Resistor_SMD:R_0805_2012Metric_Pad1.20x1.40mm_HandSolder, symbol Device:R
- removed R39: 100k, Resistor_SMD:R_0805_2012Metric_Pad1.20x1.40mm_HandSolder, symbol Device:R
- removed R40, R44, R45: 10k, Resistor_SMD:R_0805_2012Metric_Pad1.20x1.40mm_HandSolder, symbol Device:R
- removed R41: 4.7k, Resistor_SMD:R_0805_2012Metric_Pad1.20x1.40mm_HandSolder, symbol Device:R
- removed R42: 330, Resistor_SMD:R_0805_2012Metric_Pad1.20x1.40mm_HandSolder, symbol Device:R
- removed R43, R52: 22k, Resistor_SMD:R_0805_2012Metric_Pad1.20x1.40mm_HandSolder, symbol Device:R
- removed R46: 47k', Resistor_SMD:R_0805_2012Metric_Pad1.20x1.40mm_HandSolder, symbol Device:R
- removed U10: AP3031KTR, Package_TO_SOT_SMD:SOT-23-6_Handsoldering, symbol AP3031:AP3031KTR
- added C30: 2.2n, Capacitor_SMD:C_0805_2012Metric_Pad1.18x1.45mm_HandSolder, symbol Device:C
- added C31, C34: 4.7u, Capacitor_SMD:C_0805_2012Metric_Pad1.18x1.45mm_HandSolder, symbol Device:C
- added D10: B5819W, Diode_SMD:D_SOD-123, symbol Diode:MBR0540
- added L3: 10u, srn3010C-100m:IND_SRN3010C-100M, symbol Device:L
- added Q10, Q11: BSS138, Package_TO_SOT_SMD:SOT-23, symbol Transistor_FET:BSS138
- added Q18: AO3419, Package_TO_SOT_SMD:SOT-23_Handsoldering, symbol Transistor_FET:IRLML6402
- added R62, R63: 1M, Resistor_SMD:R_0805_2012Metric_Pad1.20x1.40mm_HandSolder, symbol Device:R
- added R64: 13.3, Resistor_SMD:R_0805_2012Metric_Pad1.20x1.40mm_HandSolder, symbol Device:R
- added R65: 10k, Resistor_SMD:R_0805_2012Metric_Pad1.20x1.40mm_HandSolder, symbol Device:R
- added U11: AP3031KTR, Package_TO_SOT_SMD:SOT-23-6_Handsoldering, symbol AP3031:AP3031KTR
- L1: value 22u -> [22u] 47u
- Q4: value BSS138 -> [BSS138] AO3400A
Connections:
- net 3V3: now also Q18.2 (S), R65.2
- net C-: now also Q11.3 (D), R63.1
- net COLOR_SEL: now also Q11.1 (G)
- net COLOR_SEL_INV: now also C30.1, Q10.1 (G)
- net GND: now also C30.2, C31.1, C34.1, R62.2, R63.2, R64.2, U11.2 (GND)
- net LED_ACTIVATE: now also Q18.1 (G), R65.1
- net LED_SW: now also C34.2, D10.1 (K), U11.5 (OV)
- net PWM_LED: now also U11.4 (CTRL)
- net W-: now also Q10.3 (D), R62.1
- new net: C31.2, L3.1, Q18.3 (D), U11.6 (V_{IN})
- new net: D10.2 (A), L3.2, U11.1 (SW)
- new net: Q10.2 (S), Q11.2 (S), R64.1, U11.3 (FB)
Other:
- note added: "25V"
- note added: "https://tinyurl.com/y4dphkm9"
- note added: "input capacitor"
- note added: "no need for esp pullup"
- note removed: "50V"
- note removed: "Touch Connector"
- moved on the sheet: C32, C33, C5, R13, R21, R22, R23, R24, R25, R26, R29, R30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
