File: minRead_pcb.kicad_pcb (KiCad board)
At the start: 2 copper layers, 60 x 111.3 mm, 128 parts, among them J1 USB_C_Receptacle, J2 FH34SRJ-24S-0.5SH_50_, J3 FH34SRJ-6S-0.5SH_50_, J5 Conn_01x02, J6 PPPC062LJBN-RC, J7 Micro_SD_Card, Q1 FS8205A, Q2 AO3419, Q3 AO3419, Q4 BSS138, Q5 BSS138, Q6 BSS138, Q7 AO3419, Q8 AO3419, Q9 MMBT3904, SW1 SW_Push, SW10 SW_Push, SW11 SW_Push, SW2 SW_Push, SW3 SW_Push, SW4 SW_Push, SW5 SW_Push, SW6 SW_Push, SW7 SW_Push, SW8 SW_Push, SW9 SW_Push, U1 TPD4E1U06DBVR, U2 LM27313XMF, U3 AP2112K-3.3, U4 ESP32-S3-WROOM-1, U5 DW01A, U6 TPD4E1U06DBVR, U7 MCP73832-2-OT, U8 TPD4E1U06DBVR, U9 TPD4E1U06DBVR

Commit message: updated schematic with new LED circuit, new power path, new protections, esd fix ups, etc. resetting layout, will do later
Parts:
- added C21: 1n, Capacitor_SMD:C_0805_2012Metric_Pad1.18x1.45mm_HandSolder, B.Cu at (290.9, 122.3)
- added C23: 100n, Capacitor_SMD:C_0805_2012Metric_Pad1.18x1.45mm_HandSolder, B.Cu at (290.9, 125.3)
- added C24: 2.2n, Capacitor_SMD:C_0805_2012Metric_Pad1.18x1.45mm_HandSolder, B.Cu at (290.9, 128.3)
- added C25: 1u, Capacitor_SMD:C_0805_2012Metric_Pad1.18x1.45mm_HandSolder, B.Cu at (24.0, -17.5)
- added C26: 1u, Capacitor_SMD:C_0805_2012Metric_Pad1.18x1.45mm_HandSolder, B.Cu at (24.0, -14.5)
- added C27: 2.2n, Capacitor_SMD:C_0805_2012Metric_Pad1.18x1.45mm_HandSolder, B.Cu at (161.9, 68.3)
- added C28: 2.2n, Capacitor_SMD:C_0805_2012Metric_Pad1.18x1.45mm_HandSolder, B.Cu at (161.9, 71.3)
- added D2: LED, LED_THT:LED_D3.0mm, B.Cu at (45.4, -4.65)
- added D9: BZT52C22, Diode_SMD:D_SOD-123F, B.Cu at (311.2, 148.6)
- added J4: FH34SRJ-6S-0.5SH_50_, FH34SRJ-6S-0.5SH(50):HRS_FH34SRJ-6S-0.5SH_50_, B.Cu at (161.0, 76.0)
- added Q12: MMBT3904, Package_TO_SOT_SMD:SOT-23_Handsoldering, B.Cu at (296.5, 123.3)
- added Q13: MMBT3904, Package_TO_SOT_SMD:SOT-23_Handsoldering, B.Cu at (296.5, 128.1)
- added Q14: AO3419, Package_TO_SOT_SMD:SOT-23_Handsoldering, B.Cu at (296.5, 132.8)
- added Q15: MMBT3906, Package_TO_SOT_SMD:SOT-23_Handsoldering, B.Cu at (296.5, 137.6)
- added Q16: MMBT3906, Package_TO_SOT_SMD:SOT-23_Handsoldering, B.Cu at (296.5, 142.4)
- added Q17: MMBT3904, Package_TO_SOT_SMD:SOT-23_Handsoldering, B.Cu at (296.5, 147.2)
- added Q9: BSS138, Package_TO_SOT_SMD:SOT-23, B.Cu at (305.6, 148.4)
- added R17: 1M, Resistor_SMD:R_0805_2012Metric_Pad1.20x1.40mm_HandSolder, B.Cu at (311.6, 122.2)
- added R38: 310k, Resistor_SMD:R_0805_2012Metric_Pad1.20x1.40mm_HandSolder, B.Cu at (44.7, -23.6)
- added R39: 100k, Resistor_SMD:R_0805_2012Metric_Pad1.20x1.40mm_HandSolder, B.Cu at (311.6, 128.2)
- added R41: 4.7k, Resistor_SMD:R_0805_2012Metric_Pad1.20x1.40mm_HandSolder, B.Cu at (311.6, 131.1)
- added R42: 330, Resistor_SMD:R_0805_2012Metric_Pad1.20x1.40mm_HandSolder, B.Cu at (311.6, 134.1)
- added R43: 22k, Resistor_SMD:R_0805_2012Metric_Pad1.20x1.40mm_HandSolder, B.Cu at (311.6, 137.0)
- added R44: 10k, Resistor_SMD:R_0805_2012Metric_Pad1.20x1.40mm_HandSolder, B.Cu at (311.6, 139.9)
- added R45: 10k, Resistor_SMD:R_0805_2012Metric_Pad1.20x1.40mm_HandSolder, B.Cu at (306.9, 122.2)
- added R46: 47k', Resistor_SMD:R_0805_2012Metric_Pad1.20x1.40mm_HandSolder, B.Cu at (306.9, 125.2)
- added R47: 18k, Resistor_SMD:R_0805_2012Metric_Pad1.20x1.40mm_HandSolder, B.Cu at (306.9, 128.2)
- added R48: 18k, Resistor_SMD:R_0805_2012Metric_Pad1.20x1.40mm_HandSolder, B.Cu at (306.9, 131.1)
- added R49: 1M, Resistor_SMD:R_0805_2012Metric_Pad1.20x1.40mm_HandSolder, B.Cu at (306.9, 134.1)
- added R50: 1M, Resistor_SMD:R_0805_2012Metric_Pad1.20x1.40mm_HandSolder, B.Cu at (306.9, 137.0)
- added R51: 100k, Resistor_SMD:R_0805_2012Metric_Pad1.20x1.40mm_HandSolder, B.Cu at (39.9, -8.86)
- added R52: 22k, Resistor_SMD:R_0805_2012Metric_Pad1.20x1.40mm_HandSolder, B.Cu at (302.1, 122.2)
- added R56: 1k, Resistor_SMD:R_0805_2012Metric_Pad1.20x1.40mm_HandSolder, B.Cu at (173.1, 56.1)
- added R57: 100k, Resistor_SMD:R_0805_2012Metric_Pad1.20x1.40mm_HandSolder, B.Cu at (173.1, 59.1)
- added R58: 100k, Resistor_SMD:R_0805_2012Metric_Pad1.20x1.40mm_HandSolder, B.Cu at (35.2, -17.7)
- added R59: 1k, Resistor_SMD:R_0805_2012Metric_Pad1.20x1.40mm_HandSolder, B.Cu at (35.2, -14.8)
- added R60: 100, Resistor_SMD:R_0805_2012Metric_Pad1.20x1.40mm_HandSolder, B.Cu at (173.1, 68.0)
- added R61: 100, Resistor_SMD:R_0805_2012Metric_Pad1.20x1.40mm_HandSolder, B.Cu at (173.1, 70.9)
- added U10: AP3031KTR, Package_TO_SOT_SMD:SOT-23-6_Handsoldering, B.Cu at (305.2, 143.9)
- added U2: TPS2116DRL, Package_TO_SOT_SMD:SOT-583-8, B.Cu at (19.7, -26.0)
- R37: value 82 -> 13.3
- moved C12 242.4 mm to (285.8, 163.4)
- moved D7 242.4 mm to (288.3, 173.4)
- moved L2 242.4 mm to (285.2, 168.9)
- moved Q5 242.4 mm to (289.0, 158.0)
- moved Q7 242.4 mm to (290.5, 163.4)
- moved Q9 242.4 mm to (296.5, 164.7)
- moved R37 242.4 mm to (293.8, 169.6)
- moved R39 242.4 mm to (291.0, 166.2)
- moved R40 242.4 mm to (293.2, 159.4)
- moved R41 242.4 mm to (298.2, 160.4)
- moved C9 242.4 mm to (292.6, 173.4)
- moved Q6 242.4 mm to (292.6, 156.3)
- moved J1 159.3 mm to (-40.5, 43.9)
- moved R10 159.3 mm to (-51.7, -3.51)
- moved R12 159.3 mm to (-53.7, -3.51)
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Connections:
- D7 pad 2: Net-(D7-A) -> /3031_SW
- L2 pad 2: Net-(D7-A) -> /3031_SW
- Q3 pad 1: B- -> Net-(Q3-G)
- Q5 pad 1: COOL_TOGGLE -> COLOR_SEL
- Q6 pad 1: WARM_TOGGLE -> /COLOR_SEL_INV
- Q7 pad 1: LED_PWR -> Net-(Q7-G)
- R40 pad 1: LED_PWR -> Net-(Q7-G)
- SW1 pad 2: BUTTON_ADC_2 -> Net-(R61-Pad1)
- SW2 pad 2: BUTTON_ADC_1 -> Net-(R60-Pad1)
- U4 pad 11: LED_SENSE -> unconnected-(U4-IO18-Pad11)
- U4 pad 7: COOL_TOGGLE -> unconnected-(U4-IO7-Pad7)
- U7 pad 1: CHG_STATUS -> Net-(U7-STAT)
Routing:
- net 3V3: track 243.6 -> 0.00 mm, vias 20 -> 0
- net LED_SW: track 137.9 -> 0.00 mm, vias 2 -> 0
- net W-: track 126.1 -> 0.00 mm, vias 2 -> 0
- net C-: track 123.3 -> 0.00 mm, vias 2 -> 0
- net BUTTON_ADC_2: track 94.4 -> 0.00 mm
- net ESP32_EN: track 94.2 -> 0.00 mm, vias 4 -> 0
- net P+: track 90.6 -> 0.00 mm, vias 3 -> 0
- net UNUSED_GPIO_16: track 80.8 -> 0.00 mm, vias 2 -> 0
- net UNUSED_GPIO_46: track 80.3 -> 0.00 mm, vias 2 -> 0
- net UNUSED_GPIO_15: track 79.9 -> 0.00 mm, vias 2 -> 0
- net UNUSED_GPIO_45: track 77.6 -> 0.00 mm, vias 2 -> 0
- net PWR_BUTTON: track 74.8 -> 0.00 mm, vias 1 -> 0
- net PWM_LED: track 73.7 -> 0.00 mm, vias 2 -> 0
- net RX: track 72.0 -> 0.00 mm, vias 2 -> 0
- net UNUSED_GPIO_47: track 70.8 -> 0.00 mm, vias 4 -> 0
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
Commit message: larger battery cutout
Parts:
- removed C12, C9: 4.7u, Capacitor_SMD:C_0805_2012Metric_Pad1.18x1.45mm_HandSolder
- removed C21: 1n, Capacitor_SMD:C_0805_2012Metric_Pad1.18x1.45mm_HandSolder
- removed C23: 100n, Capacitor_SMD:C_0805_2012Metric_Pad1.18x1.45mm_HandSolder
- removed C24: 2.2n, Capacitor_SMD:C_0805_2012Metric_Pad1.18x1.45mm_HandSolder
- removed C7: 0.1u, Capacitor_SMD:C_0805_2012Metric_Pad1.18x1.45mm_HandSolder
- removed CR2: TSD05CDYFR, Diode_SMD:D_SOD-323_HandSoldering
- removed the D2 at (-57.2, 36.7)
- removed D3: SMAJ30A, Diode_SMD:D_SMA
- removed D7: B5819W, Diode_SMD:D_SOD-123
- removed D8: PESD2IVN-UX, Package_TO_SOT_SMD:SOT-323_SC-70_Handsoldering
- removed D9: BZT52C22, Diode_SMD:D_SOD-123F
- removed the G*** at (99.7, 110.6)
- removed the G*** at (48.9, 110.5)
- removed the G*** at (91.4, 58.4)
- removed the G*** at (101.1, 126.9)
- removed the G*** at (60.3, 126.4)
- removed the G*** at (74.4, 80.8)
- removed J4: FH34SRJ-6S-0.5SH_50_, FH34SRJ-6S-0.5SH(50):HRS_FH34SRJ-6S-0.5SH_50_
- removed J6: PPPC062LJBN-RC, PPPC_12:CONN_PPPC062LJBN-RC_SUL
- removed L2: 22u, srn3010C-100m:IND_SRN3010C-100M
- removed Q1: FS8205A, Package_TO_SOT_SMD:SOT-23-6_Handsoldering
- removed Q12, Q13, Q9: MMBT3904, Package_TO_SOT_SMD:SOT-23_Handsoldering
- removed Q14, Q2, Q3, Q7, Q8: AO3419, Package_TO_SOT_SMD:SOT-23_Handsoldering
- removed Q15: MMBT3906, Package_TO_SOT_SMD:SOT-23_Handsoldering
- removed Q6, Q9: BSS138, Package_TO_SOT_SMD:SOT-23
- removed R16, R56: 1k, Resistor_SMD:R_0805_2012Metric_Pad1.20x1.40mm_HandSolder
- removed R17, R49, R50: 1M, Resistor_SMD:R_0805_2012Metric_Pad1.20x1.40mm_HandSolder
- removed R27: 0, Resistor_SMD:R_0805_2012Metric_Pad1.20x1.40mm_HandSolder
- removed R35: 33k, Resistor_SMD:R_0805_2012Metric_Pad1.20x1.40mm_HandSolder
- removed R36: 68k, Resistor_SMD:R_0805_2012Metric_Pad1.20x1.40mm_HandSolder
- removed R37: 13.3, Resistor_SMD:R_0805_2012Metric_Pad1.20x1.40mm_HandSolder
- removed the R38 at (-54.9, 36.7)
- removed R39, R57: 100k, Resistor_SMD:R_0805_2012Metric_Pad1.20x1.40mm_HandSolder
- removed R39, R40, R41, R44, R45: 10k, Resistor_SMD:R_0805_2012Metric_Pad1.20x1.40mm_HandSolder
- removed R41: 4.7k, Resistor_SMD:R_0805_2012Metric_Pad1.20x1.40mm_HandSolder
- removed R42: 330, Resistor_SMD:R_0805_2012Metric_Pad1.20x1.40mm_HandSolder
- removed R43, R52: 22k, Resistor_SMD:R_0805_2012Metric_Pad1.20x1.40mm_HandSolder
- removed R46: 47k', Resistor_SMD:R_0805_2012Metric_Pad1.20x1.40mm_HandSolder
- removed SW5, SW7: SW_Push, mjtp1117:MJTP1117
- removed U10: AP3031KTR, Package_TO_SOT_SMD:SOT-23-6_Handsoldering
- removed the U2 at (-84.3, 38.2)
- removed U5: DW01A, Package_TO_SOT_SMD:SOT-23-6_Handsoldering
- removed U8, U9: TPD4E1U06DBVR, Package_TO_SOT_SMD:SOT-23-6_Handsoldering
- added C29: 2.2n, Capacitor_SMD:C_0805_2012Metric_Pad1.18x1.45mm_HandSolder, B.Cu at (194.2, 27.8)
- added C30: 2n2, Capacitor_SMD:C_0805_2012Metric_Pad1.18x1.45mm_HandSolder, B.Cu at (194.2, 30.8)
- added C31: 4u7, Capacitor_SMD:C_0805_2012Metric_Pad1.18x1.45mm_HandSolder, B.Cu at (194.2, 33.8)
- added C34: 4u7, Capacitor_SMD:C_0805_2012Metric_Pad1.18x1.45mm_HandSolder, B.Cu at (194.2, 36.8)
- added D10: B5819W, Diode_SMD:D_SOD-123, B.Cu at (188.9, 42.3)
- added L3: 10u, srn3010C-100m:IND_SRN3010C-100M, B.Cu at (183.4, 38.4)
- added Q10: BSS138, Package_TO_SOT_SMD:SOT-23, B.Cu at (182.9, 28.5)
- added Q11: BSS138, Package_TO_SOT_SMD:SOT-23, B.Cu at (182.9, 33.0)
- added Q18: AO3419, Package_TO_SOT_SMD:SOT-23_Handsoldering, B.Cu at (188.6, 33.6)
- added R62: 1M, Resistor_SMD:R_0805_2012Metric_Pad1.20x1.40mm_HandSolder, B.Cu at (199.0, 27.8)
- added R63: 1M, Resistor_SMD:R_0805_2012Metric_Pad1.20x1.40mm_HandSolder, B.Cu at (199.0, 30.7)
- added R64: 13R3 1%, Resistor_SMD:R_0805_2012Metric_Pad1.20x1.40mm_HandSolder, B.Cu at (199.0, 33.7)
- added R65: 10k, Resistor_SMD:R_0805_2012Metric_Pad1.20x1.40mm_HandSolder, B.Cu at (199.0, 36.6)
- added R66: 100k, Resistor_SMD:R_0805_2012Metric_Pad1.20x1.40mm_HandSolder, B.Cu at (199.0, 39.6)
- added U11: AP3031KTR, Package_TO_SOT_SMD:SOT-23-6_Handsoldering, B.Cu at (188.9, 38.3)
- C10: value 4.7u -> 4u7 25V
- C11: value 4.7u -> 4u7
- L1: value 22u -> [22u] 47u
- Q4: value BSS138 -> [BSS138] AO3400A
- Q5: value BSS138 -> AO3419; footprint Package_TO_SOT_SMD:SOT-23 -> Package_TO_SOT_SMD:SOT-23_Handsoldering
- R14: value 3 -> 2R2
- moved Q5 163.7 mm to (188.6, 28.8), turned to 180 degrees
- moved H2 72.6 mm to (-18.4, 75.4)
- moved J7 72.6 mm to (-8.32, 82.4)
- moved R21 72.6 mm to (-20.9, 127.0)
- moved R23 72.6 mm to (-16.6, 127.0)
- moved R24 72.6 mm to (-12.4, 127.0)
- moved R26 72.6 mm to (-3.65, 119.7)
- moved R30 72.6 mm to (-3.40, 109.5)
- moved SW6 72.6 mm to (-46.6, 78.7)
- moved U1 72.6 mm to (-18.7, 88.4)
- moved U4 72.6 mm to (-19.3, 113.8)
- moved C32 72.6 mm to (-25.6, 99.5)
- moved C33 72.6 mm to (-26.6, 102.5)
- moved C36 72.6 mm to (2.59, 85.7)
- moved C37 72.6 mm to (0.59, 85.7)
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Connections:
- C1 pad 1: GND -> B-
- C10 pad 1: GND -> B-
- C13 pad 1: GND -> B-
- C14 pad 1: GND -> B-
- C15 pad 1: GND -> B-
- C16 pad 1: GND -> B-
- C17 pad 1: GND -> B-
- C18 pad 1: GND -> B-
- C19 pad 1: GND -> B-
- C2 pad 2: GND -> B-
- C20 pad 1: GND -> B-
- C22 pad 1: GND -> B-
- C25 pad 1: GND -> B-
- C26 pad 2: GND -> B-
- C27 pad 1: GND -> B-
- C28 pad 1: GND -> B-
- C3 pad 2: GND -> B-
- C32 pad 2: GND -> B-
- C33 pad 2: GND -> B-
- C36 pad 1: GND -> B-
- C37 pad 1: GND -> B-
- C4 pad 2: GND -> B-
- C5 pad 2: GND -> B-
- C6 pad 2: GND -> B-
- C8 pad 2: GND -> B-
- CR1 pad 2: GND -> B-
- D6 pad 1: GND -> B-
- H1 pad 1: GND -> B-
- H2 pad 1: GND -> B-
- H3 pad 1: GND -> B-
- H4 pad 1: GND -> B-
- J1 pad A1: GND -> B-
- J1 pad A12: GND -> B-
- J1 pad B1: GND -> B-
- J1 pad B12: GND -> B-
- J2 pad 17: GND -> B-
- J2 pad 8: GND -> B-
- J2 pad S1: GND -> B-
- J2 pad S2: GND -> B-
- J3 pad S1: GND -> B-
- J3 pad S2: GND -> B-
- J7 pad 6: GND -> B-
- J7 pad 9: GND -> B-
- Q17 pad 2: GND -> B-
- Q5 pad 1: COLOR_SEL -> Net-(Q5-G)
- Q5 pad 2: Net-(Q5-S) -> P+
- Q5 pad 3: C- -> B+
- R1 pad 1: GND -> B-
- R10 pad 2: GND -> B-
- R14 pad 1: GND -> B-
- R15 pad 1: GND -> B-
- R2 pad 2: GND -> B-
- R3 pad 2: GND -> B-
- R51 pad 2: GND -> B-
- R6 pad 2: GND -> B-
- SW1 pad 1: GND -> B-
- SW11 pad 1: GND -> B-
- SW2 pad 1: GND -> B-
- SW3 pad 1: GND -> B-
- SW4 pad 1: GND -> B-
- SW6 pad 1: GND -> B-
- SW8 pad 1: GND -> B-
- SW9 pad 1: GND -> B-
- U1 pad 2: GND -> B-
- U2 pad 1: GND -> B-
- U3 pad 2: GND -> B-
- U4 pad 1: GND -> B-
- U4 pad 36: RX -> unconnected-(U4-RXD0-Pad36)
- U4 pad 37: TX -> unconnected-(U4-TXD0-Pad37)
- U4 pad 40: GND -> B-
- U4 pad 41: GND -> B-
- U6 pad 2: GND -> B-
- U7 pad 2: GND -> B-
Routing:
- added copper zone on B.Cu, net B-
- added copper zone on F.Cu, net B-
- removed copper zone on B.Cu, net GND
- removed copper zone on F.Cu, net GND
Other:
- board size 60 x 111.3 mm -> 132.4 x 111.3 mm
- board text added: "LP284550/LP304550"
- board text removed: "Development Header"
- board text removed: "Github:"
- board text removed: "I U"
- board text removed: "Ko-Fi:"
- board text removed: "Patreon:"
- board text removed: "made with love by Ian C supported by several, including: Thank you all!"

Commit message: shaping
Parts:
- moved G*** 22.7 mm to (189.1, 123.6)
- moved J5 17.3 mm to (121.2, 34.5)
- moved R11 7.55 mm to (102.2, 58.1)
- moved SW1 7.55 mm to (101.9, 62.6)
- moved SW4 7.55 mm to (102.0, 48.6)
- moved R28 7.55 mm to (78.5, 59.5)
- moved R4 7.55 mm to (95.5, 64.2)
- moved R53 7.55 mm to (93.5, 64.4)
- moved R54 7.55 mm to (90.0, 64.4)
- moved R55 7.55 mm to (87.7, 64.4)
- moved R8 7.55 mm to (84.7, 64.4)
Other:
- outline, holes or cut-outs redrawn

Commit message: match screen size to pcb size
Parts:
- removed C28, C29: 2.2n, Capacitor_SMD:C_0805_2012Metric_Pad1.18x1.45mm_HandSolder
- removed R11: 12k, Resistor_SMD:R_0805_2012Metric_Pad1.20x1.40mm_HandSolder
- removed R28: 10k, Resistor_SMD:R_0805_2012Metric_Pad1.20x1.40mm_HandSolder
- removed R61: 100, Resistor_SMD:R_0805_2012Metric_Pad1.20x1.40mm_HandSolder
- removed SW1, SW4: SW_Push, mjtp1117:MJTP1117
- moved SW8 123.5 mm to (192.2, 166.3)
- moved SW9 123.5 mm to (180.2, 166.3)
- moved SW2 97.9 mm to (101.1, 48.7), turned to -90 degrees
- moved SW3 85.8 mm to (101.1, 62.5), turned to -90 degrees
- moved H4 17.9 mm to (115.8, 154.7)
- moved H3 15.6 mm to (33.4, 152.1)
Connections:
- U4 pad 38: BUTTON_ADC_2 -> unconnected-(U4-IO2-Pad38)
Other:
- board size 132.4 x 111.3 mm -> 134 x 110.5 mm

Commit message: add back bottom buttons
Parts:
- added C28: 2.2n, Capacitor_SMD:C_0805_2012Metric_Pad1.18x1.45mm_HandSolder, F.Cu at (183.8, 156.0)
- added C29: 2.2n, Capacitor_SMD:C_0805_2012Metric_Pad1.18x1.45mm_HandSolder, F.Cu at (183.8, 159.0)
- added R11: 12k, Resistor_SMD:R_0805_2012Metric_Pad1.20x1.40mm_HandSolder, F.Cu at (183.8, 147.1)
- added R28: 10k, Resistor_SMD:R_0805_2012Metric_Pad1.20x1.40mm_HandSolder, F.Cu at (183.8, 150.1)
- added R61: 100, Resistor_SMD:R_0805_2012Metric_Pad1.20x1.40mm_HandSolder, F.Cu at (183.8, 153.0)
- added SW1: SW_Push, mjtp1117:MJTP1117, F.Cu at (102.9, 53.8)
- added SW4: SW_Push, mjtp1117:MJTP1117, F.Cu at (172.8, 161.3)
- moved SW8 124.0 mm to (69.8, 146.6)
- moved SW9 124.0 mm to (57.8, 146.6)
- moved SW2 98.1 mm to (94.7, 146.6), turned to 180 degrees
- moved SW3 86.0 mm to (82.7, 146.6), turned to 180 degrees
- moved H4 17.9 mm to (100.5, 145.2)
- moved H3 15.6 mm to (47.5, 145.2)
Connections:
- U4 pad 38: unconnected-(U4-IO2-Pad38) -> BUTTON_ADC_2
Other:
- board size 134 x 110.5 mm -> 133.9 x 116.2 mm

Commit message: finish adding buttons
Parts:
- C28, C29, R11, R28, R61: moved to B.Cu
- moved SW4 128.8 mm to (101.9, 53.8), turned to 90 degrees
- moved SW1 14.0 mm to (101.9, 67.8)
- moved R11 0.06 mm to (183.8, 147.1), turned to 180 degrees
- moved R28 0.06 mm to (183.8, 150.1), turned to 180 degrees
- moved R61 0.06 mm to (183.8, 153.0), turned to 180 degrees
- turned C28 to 180 degrees
- turned C29 to 180 degrees
Other:
- outline, holes or cut-outs redrawn
