File: eink.kicad_pcb (KiCad board)
At the start: 2 copper layers, 62.4 x 115 mm, 114 parts, among them J1 USB_C_Receptacle, J2 FH34SRJ-24S-0.5SH_50_, J3 FH34SRJ-6S-0.5SH_50_, J5 Conn_01x02, J7 Micro_SD_Card, Q10 BSS138, Q11 BSS138, Q12 BSS138, Q18 AO3419, Q4 [BSS138] AO3400A, Q5 AO3419, Q6 AO3419, SW1 SW_Push, SW10 SW_Push, SW11 SW_Push, SW2 SW_Push, SW3 SW_Push, SW4 SW_Push, SW6 SW_Push, SW8 SW_Push, SW9 SW_Push, U1 TPD4E1U06DBVR, U11 AP3031KTR, U3 AP2112K-3.3, U4 ESP32-S3-WROOM-1, U5 74LVC1G04, U6 TPD4E1U06DBVR, U7 TP4054

Commit message: simulations
Parts:
- added C21: 1u, Capacitor_SMD:C_0805_2012Metric_Pad1.18x1.45mm_HandSolder, B.Cu at (91.0, 55.2)
- added R70: 10k, Resistor_SMD:R_0805_2012Metric_Pad1.20x1.40mm_HandSolder, B.Cu at (83.2, 56.0)
- moved C9 3.85 mm to (87.2, 55.2)
Connections:
- Q6 pad 1: USB_VBUS -> Net-(Q6-G)
Routing:
- net Net-(Q6-G): track 0.00 -> 11.8 mm
- net USB_VBUS: track 49.4 -> 56.2 mm
- net LDO_IN: track 58.3 -> 56.4 mm

Commit message: drc
Routing:
- net B-: vias 77 -> 78
Changed lines of the file:
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@@
 		(tags "LED handsolder")
 		(property "Reference" "D3"
-			(at 2 0.275 90)
+			(at 0 0.075 180)
 			(layer "B.SilkS")
 			(effects
@@
 		(tags "SOT-23-5 hand-soldering")
 		(property "Reference" "U5"
-			(at 0 2.9 0)
+			(at 0.4 0 0)
 			(layer "B.SilkS")
 			(effects
@@
 		(net "B-")
 	)
+	(via
+		(at 90.2 56.8)
+		(size 0.6)
+		(drill 0.3)
+		(layers "F.Cu" "B.Cu")
+		(free yes)
+		(net "B-")
+	)
