File: eink.kicad_sch (KiCad schematic)
At the start: 114 parts, among them J1 USB_C_Receptacle, J2 FH34SRJ-24S-0.5SH_50_, J3 FH34SRJ-6S-0.5SH_50_, J5 Conn_01x02, J7 Micro_SD_Card, Q10 BSS138, Q11 BSS138, Q12 BSS138, Q18 AO3419, Q4 [BSS138] AO3400A, Q5 AO3419, Q6 AO3419, SW1 SW_Push, SW10 SW_Push, SW11 SW_Push, SW2 SW_Push, SW3 SW_Push, SW4 SW_Push, SW6 SW_Push, SW8 SW_Push, SW9 SW_Push, U1 TPD4E1U06DBVR, U11 AP3031KTR, U3 AP2112K-3.3, U4 ESP32-S3-WROOM-1, U5 74LVC1G04, U6 TPD4E1U06DBVR, U7 TP4054

Commit message: misc
Other:
- note added: "no need for pullup floating pin since frontlight will be turned on reasonably after startup"
Changed lines of the file:
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@@
+		)
+	)
+	(text "no need for pullup floating pin since frontlight will be turned on reasonably after startup"
+		(exclude_from_sim no)
+		(at 260.35 339.598 0)
+		(effects
+			(font
+				(size 1.27 1.27)
+			)
 		)
 	)

Commit message: simulations
Parts:
- added C21: 1u, Capacitor_SMD:C_0805_2012Metric_Pad1.18x1.45mm_HandSolder, symbol Device:C
- added R70: 10k, Resistor_SMD:R_0805_2012Metric_Pad1.20x1.40mm_HandSolder, symbol Device:R
Connections:
- net GND: now also C21.2
- net USB_VBUS: now also R70.2; no longer Q6.1 (G)
- new net: C21.1, Q6.1 (G), R70.1
Other:
- note added: "10ms RC filter to prevent voltage drop See "power path" sim"
- moved on the sheet: C9, R67

Commit message: drc
Other:
- moved on the sheet: C24, U5
Changed lines of the file:
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@@
 	)
 	(junction
-		(at 256.54 311.15)
+		(at 246.38 308.61)
 		(diameter 0)
 		(color 0 0 0 0)
@@
 	(wire
 		(pts
-			(xy 256.54 302.26) (xy 256.54 311.15)
+			(xy 246.38 299.72) (xy 246.38 308.61)
 		)
 		(stroke
@@
 	(wire
 		(pts
-			(xy 256.54 311.15) (xy 256.54 312.42)
+			(xy 246.38 308.61) (xy 246.38 309.88)
 		)
 		(stroke
@@
 	)
 	(label "COLOR_SEL_INV"
-		(at 274.32 321.31 0)
+		(at 264.16 318.77 0)
 		(effects
 			(font
@@
 	(global_label "COLOR_SEL"
 		(shape input)
-		(at 246.38 321.31 180)
+		(at 236.22 318.77 180)
 		(fields_autoplaced yes)
 		(effects
@@
 		)
 		(property "Intersheetrefs" "${INTERSHEET_REFS}"
-			(at 232.8115 321.31 0)
+			(at 222.6515 318.77 0)
 			(hide yes)
 			(show_name no)
@@
 	(global_label "3V3"
 		(shape input)
-		(at 256.54 302.26 180)
+		(at 246.38 299.72 180)
 		(fields_autoplaced yes)
 		(effects
@@
 		)
 		(property "Intersheetrefs" "${INTERSHEET_REFS}"
-			(at 250.0472 302.26 0)
+			(at 239.8872 299.72 0)
 			(hide yes)
 			(show_name no)
@@
 	(symbol
 		(lib_id "power:GND")
-		(at 264.16 311.15 90)
+		(at 254 308.61 90)
 		(unit 1)
 		(body_style 1)
@@
 		(fields_autoplaced yes)
 		(property "Reference" "#PWR059"
-			(at 270.51 311.15 0)
+			(at 260.35 308.61 0)
 			(hide yes)
 			(show_name no)
@@
 		)
 		(property "Value" "GND"
-			(at 267.97 311.1499 90)
+			(at 257.81 308.6099 90)
 			(show_name no)
 			(do_not_autoplace no)
@@
 		)
 		(property "Footprint" ""
-			(at 264.16 311.15 0)
+			(at 254 308.61 0)
 			(hide yes)
 			(show_name no)
@@
 		)
 		(property "Datasheet" ""
-			(at 264.16 311.15 0)
+			(at 254 308.61 0)
 			(hide yes)
 			(show_name no)
@@
 		)
 		(property "Description" "Power symbol creates a global label with name \"GND\" , ground"
-			(at 264.16 311.15 0)
+			(at 254 308.61 0)
 			(hide yes)
 			(show_name no)
@@
 	(symbol
 		(lib_id "74xGxx:74LVC1G04")
-		(at 261.62 321.31 0)
+		(at 251.46 318.77 0)
 		(unit 1)
 		(body_style 1)
@@
 		(fields_autoplaced yes)
 		(property "Reference" "U5"
-			(at 273.05 314.8898 0)
+			(at 262.89 312.3498 0)
 			(show_name no)
 			(do_not_autoplace no)
@@
 		)
 		(property "Value" "74LVC1G04"
-			(at 273.05 317.4298 0)
+			(at 262.89 314.8898 0)
 			(show_name no)
 			(do_not_autoplace no)
@@
 		)
 		(property "Footprint" "Package_TO_SOT_SMD:SOT-23-5_HandSoldering"
-			(at 261.62 321.31 0)
+			(at 251.46 318.77 0)
 			(hide yes)
 			(show_name no)
@@
 		)
 		(property "Datasheet" "https://www.ti.com/lit/ds/symlink/sn74lvc1g04.pdf"
-			(at 261.62 321.31 0)
+			(at 251.46 318.77 0)
 			(hide yes)
 			(show_name no)
@@
 		)
 		(property "Description" "Single NOT Gate, Low-Voltage CMOS"
-			(at 261.62 321.31 0)
+			(at 251.46 318.77 0)
 			(hide yes)
 			(show_name no)
@@
 	(symbol
 		(lib_id "Device:C")
-		(at 260.35 311.15 90)
+		(at 250.19 308.61 90)
 		(unit 1)
 		(body_style 1)
@@
 		(dnp no)
 		(property "Reference" "C24"
-			(at 260.35 307.086 90)
+			(at 250.19 304.546 90)
 			(show_name no)
 			(do_not_autoplace no)
@@
 		)
 		(property "Value" "100n"
-			(at 260.35 304.546 90)
+			(at 250.19 302.006 90)
 			(show_name no)
 			(do_not_autoplace no)
@@
 		)
 		(property "Footprint" "Capacitor_SMD:C_0805_2012Metric_Pad1.18x1.45mm_HandSolder"
-			(at 264.16 310.1848 0)
+			(at 254 307.6448 0)
 			(hide yes)
 			(show_name no)
@@
 		)
 		(property "Datasheet" ""
-			(at 260.35 311.15 0)
+			(at 250.19 308.61 0)
 			(hide yes)
 			(show_name no)
@@
 		)
 		(property "Description" "Unpolarized capacitor"
-			(at 260.35 311.15 0)
+			(at 250.19 308.61 0)
 			(hide yes)
 			(show_name no)
@@
 	(symbol
 		(lib_id "power:GND")
-		(at 256.54 331.47 0)
+		(at 246.38 328.93 0)
 		(unit 1)
 		(body_style 1)
@@
 		(fields_autoplaced yes)
 		(property "Reference" "#PWR061"
-			(at 256.54 337.82 0)
+			(at 246.38 335.28 0)
 			(hide yes)
 			(show_name no)
@@
 		)
 		(property "Value" "GND"
-			(at 256.54 336.55 0)
+			(at 246.38 334.01 0)
 			(show_name no)
 			(do_not_autoplace no)
@@
 		)
 		(property "Footprint" ""
-			(at 256.54 331.47 0)
+			(at 246.38 328.93 0)
 			(hide yes)
 			(show_name no)
@@
 		)
 		(property "Datasheet" ""
-			(at 256.54 331.47 0)
+			(at 246.38 328.93 0)
 			(hide yes)
 			(show_name no)
@@
 		)
 		(property "Description" "Power symbol creates a global label with name \"GND\" , ground"
-			(at 256.54 331.47 0)
+			(at 246.38 328.93 0)
 			(hide yes)
 			(show_name no)
